Commit message: simple biped added

File: walkers/simple_biped.urdf (robot description, URDF)
Before this commit: robot simple_biped, 2 links, 1 joints
Links:
- removed link base_link
- added link right_leg, mass 2.0; collision cylinder length=0.5 radius=0.05; visual cylinder length=0.5 radius=0.05
- added link torso, mass 5.0; collision box size=0.2 0.1 0.3; visual box size=0.2 0.1 0.3
- link left_leg: mass None -> 2.0; geometry collision cylinder length=0.5 radius=0.05; visual cylinder length=0.5 radius=0.05
Joints:
- removed joint hip_joint
- added joint left_hip_joint: type revolute, parent torso, child left_leg, origin xyz=0.1 0 -0.15 rpy=0 0 0, axis 1 0 0, limit lower=-1.57 upper=1.57 effort=20 velocity=2.0
- added joint right_hip_joint: type revolute, parent torso, child right_leg, origin xyz=-0.1 0 -0.15 rpy=0 0 0, axis 1 0 0, limit lower=-1.57 upper=1.57 effort=20 velocity=2.0

Commit message: added knees

File: walkers/simple_biped.urdf (robot description, URDF)
Before this commit: robot simple_biped, 3 links, 2 joints
Links:
- removed link left_leg
- removed link right_leg
- added link left_lower_leg, mass 1.0; collision cylinder length=0.3 radius=0.04; visual cylinder length=0.3 radius=0.04
- added link left_upper_leg, mass 1.5; collision cylinder length=0.3 radius=0.05; visual cylinder length=0.3 radius=0.05
- added link right_lower_leg, mass 1.0; collision cylinder length=0.3 radius=0.04; visual cylinder length=0.3 radius=0.04
- added link right_upper_leg, mass 1.5; collision cylinder length=0.3 radius=0.05; visual cylinder length=0.3 radius=0.05
Joints:
- added joint left_knee_joint: type revolute, parent left_upper_leg, child left_lower_leg, origin xyz=0 0 -0.3 rpy=0 0 0, axis 1 0 0, limit lower=0 upper=2.0 effort=20 velocity=2.0
- added joint right_knee_joint: type revolute, parent right_upper_leg, child right_lower_leg, origin xyz=0 0 -0.3 rpy=0 0 0, axis 1 0 0, limit lower=0 upper=2.0 effort=20 velocity=2.0
- joint left_hip_joint: child left_leg -> left_upper_leg
- joint right_hip_joint: child right_leg -> right_upper_leg
